File: HW/arduino_based_cdc_emulator/atmegax8_with_F6188/atmegax8_with_bluetooth.kicad_pcb (KiCad board)
At the start: 2 copper layers, 41.4 x 36.1 mm, 75 parts, among them IC1 ATMEGA88-A, J1 Ant, J2 TMS, J3 TCK, J4 TDO, J5 TDI, P1 CONN_10, P2 SPI, P3 CONN_4, P4 SERIAL, P5 LM7805, U1 AP1117, U2 F-6188, U3 TL072, U4 MAX809, U5 MAX809, Y1 16MHz

Commit message: fixes in HW for F6188
Parts:
- R20, R21, R23, R8: value 22k -> 2k2
- turned C20 to 0 degrees
- turned C6 to 0 degrees
Connections:
- C20 pad 1: /BTOUTL -> Net-(C20-Pad1)
- C20 pad 2: Net-(C20-Pad2) -> /BTOUTL
- C6 pad 1: /BTOUTR -> Net-(C6-Pad1)
- C6 pad 2: Net-(C6-Pad2) -> /BTOUTR
- R21 pad 2: Net-(C20-Pad2) -> Net-(C20-Pad1)
- R8 pad 2: Net-(C6-Pad2) -> Net-(C6-Pad1)
Routing:
- net Net-(C20-Pad2): track 4.49 -> 0.00 mm
- net Net-(C20-Pad1): track 0.00 -> 4.49 mm
- net Net-(C6-Pad2): track 4.27 -> 0.00 mm
- net Net-(C6-Pad1): track 0.00 -> 4.27 mm

Commit message: correct value for mic resistors
Parts:
- R25: value 1k -> 2k
- R27: value 1k -> 2k(3k9)
Changed lines of the file:
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@@
       (effects (font (size 1 1) (thickness 0.15)) (justify mirror))
     )
-    (fp_text value "1k" (at 0 -1.75 90) (layer "B.Fab")
+    (fp_text value "2k" (at 0 -1.75 90) (layer "B.Fab")
       (effects (font (size 1 1) (thickness 0.15)) (justify mirror))
     )
@@
       (effects (font (size 1 1) (thickness 0.15)) (justify mirror))
     )
-    (fp_text value "1k" (at 0 -2.1 90) (layer "B.Fab")
-      (effects (font (size 1 1) (thickness 0.15)) (justify mirror))
-    )
+    (fp_text value "2k(3k9)" (at 0 -2.1 90) (layer "B.Fab")
+      (effects (font (size 1 1) (thickness 0.15)) (justify mirror))
+    )
